File: ENC_SW_Frontpanel.sch (EAGLE design)
At the start: 11 parts, among them SW1 SPDT

Commit message: Enlarged holes for switch; redid SW-ENC-Frontpanel
Now switch and rotary encoder are 0.75" separated.
Connections:
- net ENC_A: no longer R3.P$1
- net ENC_B: no longer R4.P$2
- net N$4: now also R4.P$2
- net N$5: now also R3.P$1
Other:
- moved on the sheet: R4
